File: kicad/dac.kicad_sch (KiCad schematic)
At the start: 20 parts, among them J1 USB_C_Receptacle_USB2.0, J2 AudioJack3, J3 Conn_01x03, J4 Conn_01x03, P1 Conn_WallPlug_Earth, T1 Transformer_SP_2S, U1 PCM2902, Y1 12MHz

Commit message: added mono amplifier and tvs diodes
Parts:
- added C1, C7: C, symbol Device:C
- added C10: 30pF, symbol Device:C
- added C2: 1u, symbol Device:C
- added C5, C6: 10-33pF, symbol Device:C
- added D2, D3: D_TVS, symbol Device:D_TVS
- added I1: 2mA, symbol Simulation_SPICE:IDC
- added I2: 10mA, symbol Simulation_SPICE:IDC
- added Q1, Q4, Q5, Q6, Q8: NPN, symbol Simulation_SPICE:NPN
- added Q2, Q3, Q7, Q9: PNP, symbol Simulation_SPICE:PNP
- added R1: 4.7k, symbol Device:R
- added R11: 20k, symbol Device:R
- added R12, R15: 1k, symbol Device:R
- added R13, R14: 234, symbol Device:R
- added R16: 10k, symbol Device:R
- added R17: 1k2, symbol Device:R
- added R18: 518, symbol Device:R
- added R19, R5, R6: 22, symbol Device:R
- added R2: 100, symbol Device:R
- added R20, R21: 33, symbol Device:R
- added R22, R23: 330m, symbol Device:R
- added R3: 3.2k, symbol Device:R
- added R4: 1k5, symbol Device:R
- added TH1: NTC, symbol Device:Thermistor_NTC
- added U1: SSR, OptoDevice:Finder_34.81, symbol Relay_SolidState:34.81-8240
- renumbered C1 to C3, C2 to C4, C3 to C8, C4 to C9, D2 to D1, D1 to D4, J3 to J2, J4 to J3, J2 to J4, R3 to R7, R1 to R8, R2 to R9, U1 to U2
Connections:
- net GND is gone; now on net GNDA: J4.S
- net +36V: now also C3.1, R8.1, I1.1, I2.1, Q6.1 (C), Q8.1 (C), R1.1, R3.1
- net -36V: now also Q3.1 (C), Q7.1 (C), Q9.1 (C), R12.1, R19.1
- net GNDA: now also D1.1 (A1), J1.A1 (GND), J1.A12 (GND), J1.B1 (GND), J1.B12 (GND), J1.S1 (SHIELD), U2.11 (AGNDC), U2.18 (AGNDP), U2.22 (AGNDX), U2.26 (DGND), U2.4 (DGNDU), C1.2, C2.2, C5.2, C6.2, D2.1 (A1), D3.1 (A1), Q1.3 (E), R11.1, R15.1, R2.2
- net at T1.1 (IN+): now also TH1.2, U1.14; no longer P1.1 (AC_P)
- net at J1.A4 (VBUS), J1.A9 (VBUS), J1.B4 (VBUS)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: now also U2.3 (VBUS), C2.1, D3.2 (A2), R4.2
- net at J1.A6 (D+): now also D1.2 (A2), J1.B6 (D+), R4.1, R6.1
- net at J1.A7 (D-): now also J1.B7 (D-), D2.2 (A2), R5.1
- net at U2.1 (D+): now also R6.2
- net at U2.2 (D-): now also R5.2
- net at R7.2, U2.20 (XTO), Y1.1: now also C6.1
- net at R7.1, U2.21 (XTI), Y1.2: now also C5.1
- net OUT_R: now reaches J4.R
- net OUT_L: now reaches J4.T
- net OUT_L: now also R16.2, R20.1, R21.2, R22.1, R23.2
- new net: Q1.1 (C), U1.A2
- new net: C1.1, Q1.2 (B), R1.2, R2.1
- new net: Q6.3 (E), Q8.2 (B), R20.2
- new net: Q3.2 (B), R15.2, R16.1
- new net: C7.2, Q2.2 (B), R11.2
- new net: Q8.3 (E), R22.2
- new net: Q7.3 (E), Q9.2 (B), R21.1
- new net: P1.1 (AC_P), TH1.1, U1.11
- new net: Q9.3 (E), R23.1
- new net: Q4.2 (B), R17.1, R18.2
- new net: I2.2, Q4.1 (C), Q6.2 (B), R17.2
- new net: C10.2, Q4.3 (E), Q5.1 (C), Q7.2 (B), R18.1
- new net: C10.1, Q2.1 (C), Q5.2 (B), R12.2
- new net: Q5.3 (E), R19.2
- new net: I1.2, R13.2, R14.1
- new net: Q2.3 (E), R13.1
- new net: R3.2, U1.A1
- new net: Q3.3 (E), R14.2
- new net IN_L: C7.1
- no-connect marks 6 -> 10
Other:
- note added: "wrong symbol"
- note removed: "probably wrong symbol"
- moved on the sheet: C3, C4, C8, C9, D4, F1, F2, J1, J2, J3, P1, R7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

Commit message: commit
Parts:
- removed C1, C7: C, symbol Device:C
- removed C10: 30pF, symbol Device:C
- removed C6: 10-33pF, symbol Device:C
- removed HS1: Heatsink_Pad, symbol Mechanical:Heatsink_Pad
- removed I1: 2mA, symbol Simulation_SPICE:IDC
- removed I2: 10mA, symbol Simulation_SPICE:IDC
- removed Q1, Q4, Q5, Q6, Q8: NPN, symbol Simulation_SPICE:NPN
- removed Q2, Q3, Q7, Q9: PNP, symbol Simulation_SPICE:PNP
- removed R1: 4.7k, symbol Device:R
- removed R11: 20k, symbol Device:R
- removed R12, R15: 1k, symbol Device:R
- removed R13, R14: 234, symbol Device:R
- removed R16: 10k, symbol Device:R
- removed R17: 1k2, symbol Device:R
- removed R18: 518, symbol Device:R
- removed R19: 22, symbol Device:R
- removed R2: 100, symbol Device:R
- removed R20, R21: 33, symbol Device:R
- removed R22, R23: 330m, symbol Device:R
- removed R3: 3.2k, symbol Device:R
- removed TH1: NTC, symbol Device:Thermistor_NTC
- removed U1: SSR, OptoDevice:Finder_34.81, symbol Relay_SolidState:34.81-8240
- removed U2: PCM2902, Package_SO:SSOP-28_5.3x10.2mm_P0.65mm, symbol Audio:PCM2902
- removed Y1: 12MHz, symbol Device:Crystal
- added C3, C8, C9: 1u, Capacitor_SMD:C_0805_2012Metric_Pad1.18x1.45mm_HandSolder, symbol Device:C
- added C4: 10u, symbol Device:C_Polarized
- added D1, D8: D_TVS, symbol Device:D_TVS
- added D6, D7: 40V, symbol Device:D_TVS
- added H1, H2, H3, H4: MountingHole_Pad, symbol Mechanical:MountingHole_Pad
- added H5: ~, symbol library:Knob
- added R4: 5.1k, Resistor_SMD:R_0805_2012Metric_Pad1.20x1.40mm_HandSolder, symbol Device:R
- added R8: 1k5, Resistor_SMD:R_0805_2012Metric_Pad1.20x1.40mm_HandSolder, symbol Device:R
- added U2: PCM2704/4C/5/5C, Package_SO:SSOP-28_5.3x10.2mm_P0.65mm, symbol library:PCM2704/4C/5/5C
- added Y1: 12MHz±0.05%, symbol Device:Resonator
- C2: footprint (none) -> Capacitor_SMD:C_0805_2012Metric_Pad1.18x1.45mm_HandSolder
- C5: value 10-33pF -> 1u; footprint (none) -> Capacitor_SMD:C_0805_2012Metric_Pad1.18x1.45mm_HandSolder
- J1: footprint (none) -> Connector_USB:USB_C_Receptacle_GCT_USB4085; Digikey (none) -> 2073-USB4085-GF-ACT-ND; Digikey-Alternative (none) -> SMD Variant: 2073-USB4105-GF-A-120CT-ND
- J4: Digikey (none) -> 889-1818-ND
- R10: renamed from R9; footprint (none) -> Resistor_THT:R_Axial_DIN0207_L6.3mm_D2.5mm_P10.16mm_Horizontal
- R11: renamed from R7; footprint (none) -> Resistor_SMD:R_0805_2012Metric_Pad1.20x1.40mm_HandSolder
- R5: renamed from R4; footprint (none) -> Resistor_SMD:R_0805_2012Metric_Pad1.20x1.40mm_HandSolder
- R6: renamed from R5; footprint (none) -> Resistor_SMD:R_0805_2012Metric_Pad1.20x1.40mm_HandSolder
- R7: renamed from R6; footprint (none) -> Resistor_SMD:R_0805_2012Metric_Pad1.20x1.40mm_HandSolder
- R9: renamed from R8; footprint (none) -> Resistor_THT:R_Axial_DIN0207_L6.3mm_D2.5mm_P10.16mm_Horizontal
- T1: Digikey (none) -> 237-1328-ND
- renumbered C8 to C10, C9 to C11, C3 to C6, C4 to C7, D1 to D2, D2 to D3, D3 to D4, D4 to D5
Connections:
- net GNDA: now also C2.1, C3.1, C4.2, D1.2 (A2), D8.2 (A2), R4.2, U2.11 (ZGND), U2.19 (PGND), U2.21 (HOST), U2.22 (HID0), U2.23 (HID1), U2.24 (HID2), U2.6 (DGND), Y1.2; no longer C2.2, D2.1 (A1), D3.1 (A1), D4.1 (A1), J1.S1 (SHIELD)
- net IN_L: now also U2.14 (VOUTL)
- net OUT_L: now also D7.2 (A2)
- net OUT_R: now also D6.2 (A2)
- net at J1.A4 (VBUS), J1.A9 (VBUS), J1.B4 (VBUS)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: no longer C2.1, D4.2 (A2), R5.2
- net at T1.1 (IN+): now also P1.1 (AC_P)
- net at J1.A5 (CC1): now also J1.B5 (CC2), R4.1
- net at R11.2: now also U2.1 (XTO), Y1.1
- net at R7.2: now also U2.9 (D+)
- net at R6.2: now also U2.8 (D-)
- net at R11.1: now also U2.28 (XTI), Y1.3; no longer C5.1
- net Earth: now reaches P1.3 (EARTH)
- net Earth: now also D2.1 (A1), D3.1 (A1), D4.1 (A1), J1.S1 (SHIELD), D1.1 (A1), D6.1 (A1), D7.1 (A1), D8.1 (A1)
- new net: C8.1, U2.17 (AGNDR)
- new net: C8.2, U2.16 (VccR)
- new net: C3.2, U2.20 (Vccp)
- new net: C9.1, U2.12 (AGNDL)
- new net: C9.2, U2.13 (VccL)
- new net: C4.1, U2.18 (Vcom)
- new net: R8.1, U2.3 (DT)
- new net: C5.1, U2.7 (Vdd)
- new net: U2.25 (TEST1), U2.26 (TEST0)
- new net GNDPWR: H1.1, H2.1, H3.1, H4.1
- new net IN_R: U2.15 (VOUTR)
- no-connect marks 10 -> 11
Other:
- added sheet amplifier_left (amplifier_left.kicad_sch)
- added sheet amplifier_right (amplifier_right.kicad_sch)
- note added: "dac ic"
- note added: "filtering for input and vas stage missing"
- note added: "hardware"
- note added: "output"
- note added: "stereo amplifier"
- note added: "use input module"
- note removed: "amplifier"
- note removed: "dac"
- note removed: "wrong symbol"
- moved on the sheet: C10, C11, C6, C7, D5, F1, F2, J2, J3, P1, R10, R11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
