File: kicad/dac/dac.kicad_pcb (KiCad board)
At the start: 4 copper layers, 90 x 99 mm, 128 parts, among them J1 Conn_02x08_Odd_Even, Q1 MMBT5551, Q10 MMBT5551, Q11 MMBT5401, Q12 2SC4511, Q13 2SA1725, Q14 BCM53DS, Q15 BCM53DS, Q16 BCM56DS, Q17 MMBT5551, Q18 BCM53DS, Q19 MMBT5551, Q2 BCM53DS, Q20 MMBT5551, Q21 MMBT5551, Q22 MMBT5401, Q23 2SC4511, Q24 2SA1725, Q3 BCM53DS, Q4 BCM53DS, Q5 BCM56DS, Q6 MMBT5551, Q7 BCM53DS, Q8 MMBT5551, Q9 MMBT5551, U1 CS4349

Commit message: commit
Parts:
- removed D10, D9: ~, Package_TO_SOT_SMD:SOT-23-3
- removed Q21: MMBT5551, Package_TO_SOT_SMD:SOT-23-3
- removed Q22: MMBT5401, Package_TO_SOT_SMD:SOT-23-3
- removed Q23: 2SC4511, Package_TO_SOT_THT:TO-220F-3_Vertical
- removed Q24: 2SA1725, Package_TO_SOT_THT:TO-220F-3_Vertical
- added C28: 10u, Capacitor_SMD:C_1206_3216Metric_Pad1.33x1.80mm_HandSolder, F.Cu at (121.6, 90.3)
- added C29: 30p, Capacitor_SMD:C_1206_3216Metric_Pad1.33x1.80mm_HandSolder, F.Cu at (121.6, 93.7)
- added C30: 10u, Capacitor_SMD:C_1206_3216Metric_Pad1.33x1.80mm_HandSolder, F.Cu at (121.6, 97.0)
- added C31: 10u, Capacitor_SMD:C_1206_3216Metric_Pad1.33x1.80mm_HandSolder, F.Cu at (121.6, 100.4)
- added C32: 10u, Capacitor_SMD:C_1206_3216Metric_Pad1.33x1.80mm_HandSolder, F.Cu at (121.6, 103.7)
- added C33: 20n, Capacitor_SMD:C_1206_3216Metric_Pad1.33x1.80mm_HandSolder, F.Cu at (121.6, 107.1)
- added K1: Relay, Relay_SMD:Relay_DPDT_Omron_G6K-2F-Y, F.Cu at (123.7, 144.0)
- added R37: 68, Resistor_SMD:R_1206_3216Metric_Pad1.30x1.75mm_HandSolder, F.Cu at (127.6, 83.6)
- added R60: 16, Resistor_SMD:R_1206_3216Metric_Pad1.30x1.75mm_HandSolder, F.Cu at (139.5, 100.0)
- C10: value 3u3 -> 100n; footprint Capacitor_THT:C_Rect_L7.2mm_W7.2mm_P5.00mm_FKS2_FKP2_MKS2_MKP2 -> Capacitor_SMD:C_1206_3216Metric_Pad1.33x1.80mm_HandSolder
- C11: value 100n -> 10u
- C14, C15: value 20n -> 10u
- C16, C25: value 10u -> 20n
- C17, C26: value 10u -> 3u3; footprint Capacitor_SMD:C_1206_3216Metric_Pad1.33x1.80mm_HandSolder -> Capacitor_THT:C_Rect_L7.2mm_W7.2mm_P5.00mm_FKS2_FKP2_MKS2_MKP2
- C18, C23: value 3u3 -> 10u; footprint Capacitor_THT:C_Rect_L7.2mm_W7.2mm_P5.00mm_FKS2_FKP2_MKS2_MKP2 -> Capacitor_SMD:C_1206_3216Metric_Pad1.33x1.80mm_HandSolder
- C19: value 30p -> 10u
- C20: value 10u -> 30p
- C24: value 30p -> 20n
- C5: value 3u3 -> 470u; footprint Capacitor_SMD:C_1206_3216Metric_Pad1.33x1.80mm_HandSolder -> Capacitor_THT:CP_Radial_D10.0mm_P5.00mm
- C6: value 10u -> 470u; footprint Capacitor_SMD:C_1206_3216Metric_Pad1.33x1.80mm_HandSolder -> Capacitor_THT:CP_Radial_D10.0mm_P5.00mm
- C7: value 470u -> 3u3; footprint Capacitor_THT:CP_Radial_D10.0mm_P5.00mm -> Capacitor_SMD:C_1206_3216Metric_Pad1.33x1.80mm_HandSolder
- C8: value 470u -> 3u3; footprint Capacitor_THT:CP_Radial_D10.0mm_P5.00mm -> Capacitor_THT:C_Rect_L7.2mm_W7.2mm_P5.00mm_FKS2_FKP2_MKS2_MKP2
- D1: value ~ -> D; footprint Package_TO_SOT_SMD:SOT-23-3 -> Diode_SMD:D_SOD-323_HandSoldering
- Q10, Q19: value MMBT5551 -> 2SC4511; footprint Package_TO_SOT_SMD:SOT-23-3 -> Package_TO_SOT_THT:TO-220F-3_Vertical
- Q11: value MMBT5401 -> 2SA1725; footprint Package_TO_SOT_SMD:SOT-23-3 -> Package_TO_SOT_THT:TO-220F-3_Vertical
- Q12: value 2SC4511 -> BCM53DS; footprint Package_TO_SOT_THT:TO-220F-3_Vertical -> Package_SO:SC-74-6_1.5x2.9mm_P0.95mm
- Q13: value 2SA1725 -> BCM53DS; footprint Package_TO_SOT_THT:TO-220F-3_Vertical -> Package_SO:SC-74-6_1.5x2.9mm_P0.95mm
- Q14, Q15: value BCM53DS -> BCM56DS
- Q16: value BCM56DS -> BCM53DS
- Q17, Q6, Q8: value MMBT5551 -> BCM56DS; footprint Package_TO_SOT_SMD:SOT-23-3 -> Package_SO:SC-74-6_1.5x2.9mm_P0.95mm
- Q20: value MMBT5551 -> 2SA1725; footprint Package_TO_SOT_SMD:SOT-23-3 -> Package_TO_SOT_THT:TO-220F-3_Vertical
- Q9: value MMBT5551 -> BCM53DS; footprint Package_TO_SOT_SMD:SOT-23-3 -> Package_SO:SC-74-6_1.5x2.9mm_P0.95mm
- R10: value 10k -> 100k
- R11, R12: value 16 -> 10k
- R13: value 2 -> 68
- R14: value 2 -> 27k
- R15, R38, R48: value 20k -> 27k; footprint Resistor_THT:R_Axial_DIN0207_L6.3mm_D2.5mm_P10.16mm_Horizontal -> Resistor_SMD:R_1206_3216Metric_Pad1.30x1.75mm_HandSolder
- R16: value 27k -> 430
- R18, R29: value 430 -> 68
- R19: value 68 -> 680
- R2, R3: value 100k -> 10k
- R20: value 680 -> 68
- R21: value 68 -> 430
- R23: value 430 -> 2k2
- R24: value 2k5 -> 27k; footprint Resistor_THT:R_Axial_DIN0207_L6.3mm_D2.5mm_P10.16mm_Horizontal -> Resistor_SMD:R_1206_3216Metric_Pad1.30x1.75mm_HandSolder
- R25: value 20k -> 2k2; footprint Resistor_THT:R_Axial_DIN0207_L6.3mm_D2.5mm_P10.16mm_Horizontal -> Resistor_SMD:R_1206_3216Metric_Pad1.30x1.75mm_HandSolder
- R26: value 2k2 -> 27k
- R27: value 27k -> 2k2
- R28: value 2k2 -> 430
- R30: value 68 -> 12
- R31: value 12 -> 22
- R32: value 22 -> 33
- R34: value 33 -> 2; footprint Resistor_SMD:R_1206_3216Metric_Pad1.30x1.75mm_HandSolder -> Resistor_THT:R_Axial_DIN0614_L14.3mm_D5.7mm_P20.32mm_Horizontal
- R35, R58, R59: value 1 -> 2
- R36: value 1 -> 16; footprint Resistor_THT:R_Axial_DIN0614_L14.3mm_D5.7mm_P20.32mm_Horizontal -> Resistor_SMD:R_1206_3216Metric_Pad1.30x1.75mm_HandSolder
- R4, R5: value 16 -> 100k
- R47: value 2k5 -> 2k2; footprint Resistor_THT:R_Axial_DIN0207_L6.3mm_D2.5mm_P10.16mm_Horizontal -> Resistor_SMD:R_1206_3216Metric_Pad1.30x1.75mm_HandSolder
- R6, R7: value 10k -> 16
- R8: value 100k -> 2
- R9: value 10k -> 2
- moved Q20 157.5 mm to (159.9, 106.5)
- moved Q19 157.5 mm to (159.9, 100.3)
- moved R58 137.7 mm to (144.6, 85.6)
- moved R59 137.7 mm to (144.6, 92.8)
- moved R48 128.6 mm to (133.5, 93.5)
- moved R47 128.5 mm to (133.5, 90.2)
- moved R38 122.5 mm to (127.6, 86.9)
- moved Q17 114.0 mm to (116.0, 106.4)
- moved HS2 113.7 mm to (135.1, 68.7)
- moved RV5 113.5 mm to (153.0, 100.3)
- moved RV4 113.5 mm to (146.0, 100.3)
- moved R36 108.3 mm to (108.4, 73.5)
- moved D1 106.9 mm to (132.9, 156.6)
- moved C26 104.9 mm to (144.3, 108.7)
- moved R8 99.8 mm to (139.2, 149.0)
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Connections:
- net /amplifier_left/CM renamed /amplifier_left/CM_L
- net Net-(U1-VBIAS) renamed /VBIAS
- C1 pad 1: GND -> VBUS
- C1 pad 2: VBUS -> GND
- C10 pad 1: -25V -> /VD_FILT
- C11 pad 1: Net-(U1-VD_FILT) -> /VD_FILT
- C12 pad 1: /DC_LP_L -> /AMP_L
- C12 pad 2: GND -> /PROT_ARC_L
- C13 pad 1: /DC_LP_R -> /AMP_R
- C13 pad 2: GND -> /PROT_ARC_R
- C14 pad 1: GND -> /DC_LP_L
- C14 pad 2: Net-(C14-Pad2) -> GND
- C15 pad 1: GND -> /DC_LP_R
- C15 pad 2: Net-(C15-Pad2) -> GND
- C16 pad 1: /AMP_L -> GND
- C17 pad 1: /AMP_R -> Net-(C16-Pad2)
- C18 pad 1: Net-(C18-Pad1) -> -20Vreg
- C18 pad 2: Net-(Q3A-B) -> GND
- C19 pad 1: Net-(Q3A-C) -> +20Vreg
- C19 pad 2: /amplifier_left/V_{bias}- -> GND
- C2 pad 1: GND -> VBUS
- C2 pad 2: VBUS -> GND
- C20 pad 1: /amplifier_left/V_{bias}+ -> /amplifier_left/IPS_L
- C20 pad 2: /amplifier_left/V_{bias}- -> /amplifier_left/V_{bias}-_L
- C21 pad 1: +20Vreg -> -20Vreg
- C22 pad 1: GND -> +20Vreg
- C22 pad 2: -20Vreg -> GND
- C23 pad 1: Net-(C23-Pad1) -> /amplifier_left/V_{bias}+_L
- C23 pad 2: Net-(Q14A-B) -> /amplifier_left/V_{bias}-_L
- C24 pad 1: Net-(Q14A-C) -> GND
- C24 pad 2: /amplifier_right/V_{bias}- -> /amplifier_left/ZOBEL_L
- C25 pad 1: /amplifier_right/V_{bias}+ -> GND
- C25 pad 2: /amplifier_right/V_{bias}- -> Net-(C25-Pad2)
- C26 pad 1: +20Vreg -> Net-(C25-Pad2)
- C26 pad 2: GND -> Net-(C26-Pad2)
- C27 pad 1: GND -> -20Vreg
- C27 pad 2: -20Vreg -> GND
- C5 pad 1: Net-(U1-VQ) -> +25V
- C6 pad 1: Net-(U1-VD_FILT) -> GND
- C6 pad 2: GND -> -25V
- C7 pad 1: +25V -> /VQ
- C8 pad 2: -25V -> +25V
- C9 pad 1: GND -> -25V
- C9 pad 2: +25V -> GND
- D1 pad 1: Net-(D1-A) -> /RLY+
- D1 pad 2: Net-(D1-C) -> /RLY-
- D2 pad 1: Net-(D1-A) -> Net-(D2-A)
- D2 pad 2: Net-(D1-C) -> /DC_LP_L
- D2 pad 3: /DC_LP_R -> Net-(D2-K)
- D3 pad 1: Net-(D1-A) -> Net-(D2-A)
- D3 pad 2: Net-(D1-C) -> /DC_LP_R
- D3 pad 3: GND -> Net-(D2-K)
- D4 pad 1: -25V -> Net-(D2-A)
- D4 pad 2: +25V -> GND
- D4 pad 3: /AMP_R -> Net-(D2-K)
- D5 pad 2: +25V -> /OUT_R
- D5 pad 3: /AMP_L -> +25V
- D6 pad 1: Net-(D6-A) -> -25V
- D6 pad 2: Net-(D6-C) -> /OUT_L
- D6 pad 3: Net-(D6-A) -> +25V
- D7 pad 1: -25V -> /amplifier_left/V_{bias}-_L
- D7 pad 2: +25V -> /AMP_L
- D7 pad 3: /OUT_R -> /amplifier_left/V_{bias}+_L
- D8 pad 1: -25V -> /amplifier_right/V_{bias}-_R
- D8 pad 2: +25V -> /AMP_R
- D8 pad 3: /OUT_L -> /amplifier_right/V_{bias}+_R
- Q1 pad 1: Net-(D1-C) -> Net-(D2-K)
- Q10 pad 1: /amplifier_left/V_{bias}+ -> /amplifier_left/V_{OPS}+_L
- Q10 pad 2: /amplifier_left/V_{OPS}+ -> +25V
- Q10 pad 3: +25V -> /amplifier_left/V_{q}+_L
- Q11 pad 1: /amplifier_left/V_{bias}- -> /amplifier_left/V_{OPS}-_L
- Q11 pad 2: /amplifier_left/V_{OPS}- -> -25V
- Q11 pad 3: -25V -> /amplifier_left/V_{q}-_L
- Q12 pad 1: /amplifier_left/V_{OPS}+ -> /amplifier_right/INPUT_R
- Q12 pad 2: +25V -> /amplifier_right/FB_L
- Q12 pad 3: /amplifier_left/V_{q}+ -> /amplifier_right/CM_R
- Q13 pad 1: /amplifier_left/V_{OPS}- -> Net-(Q13A-B)
- Q13 pad 2: -25V -> Net-(Q13A-C)
- Q13 pad 3: /amplifier_left/V_{q}- -> /amplifier_right/CC_IPS_R
- Q14 pad 1: Net-(Q14A-B) -> /amplifier_right/CM_R
- Q14 pad 2: /amplifier_right/FB -> /amplifier_right/CM_R
- Q14 pad 3: /amplifier_right/CM -> /amplifier_right/CM_R
- Q14 pad 6: Net-(Q14A-C) -> /amplifier_right/IPS_R
- Q15 pad 1: Net-(Q15A-B) -> /amplifier_right/IPS_R
- Q15 pad 2: Net-(Q15A-C) -> /amplifier_right/VAS_DARL_R
- Q15 pad 3: /amplifier_right/CC_IPS -> /amplifier_right/V_{bias}-_R
- Q15 pad 4: Net-(Q15A-B) -> Net-(Q15B-E)
- Q15 pad 5: +20Vreg -> /amplifier_right/VAS_DARL_R
- Q15 pad 6: Net-(Q15A-C) -> GND
- Q16 pad 1: /amplifier_right/CM -> Net-(Q16A-B)
- Q16 pad 2: /amplifier_right/CM -> Net-(Q16A-C)
- Q16 pad 3: /amplifier_right/CM -> /amplifier_right/CC_VAS_R
- Q16 pad 4: Net-(Q16B-E) -> Net-(Q16A-B)
- Q16 pad 5: Net-(Q16A-E) -> +20Vreg
- Q16 pad 6: Net-(Q14A-C) -> Net-(Q16A-C)
- Q17 pad 1: Net-(Q14A-C) -> /amplifier_right/V_{bias}B_R
- Q17 pad 2: Net-(Q17-E) -> /amplifier_right/V_{bias}+_R
- Q17 pad 3: GND -> +25V
- Q18 pad 1: Net-(Q18A-B) -> /amplifier_right/V_{bias}-_R
- Q18 pad 2: Net-(Q18A-C) -> -25V
- Q18 pad 3: /amplifier_right/CC_VAS -> -25V
- Q18 pad 4: Net-(Q18A-B) -> -25V
- Q18 pad 5: +20Vreg -> /amplifier_right/V_{OPS}-_R
- Q18 pad 6: Net-(Q18A-C) -> -25V
- Q19 pad 1: /amplifier_right/V_{bias}B -> /amplifier_right/V_{OPS}+_R
- Q19 pad 2: /amplifier_right/V_{bias}- -> +25V
- Q19 pad 3: /amplifier_right/V_{bias}+ -> /amplifier_right/V_{q}+_R
- Q2 pad 2: Net-(D1-A) -> Net-(D2-A)
- Q20 pad 1: Net-(Q17-E) -> /amplifier_right/V_{OPS}-_R
- Q20 pad 2: Net-(Q20-E) -> -25V
- Q20 pad 3: /amplifier_right/V_{bias}- -> /amplifier_right/V_{q}-_R
- Q3 pad 1: Net-(Q3A-B) -> /amplifier_left/INPUT_L
- Q3 pad 2: /amplifier_left/FB -> /amplifier_left/FB_L
- Q3 pad 6: Net-(Q3A-C) -> /amplifier_left/IPS_L
- Q4 pad 3: /amplifier_left/CC_IPS -> /amplifier_left/CC_IPS_L
- Q5 pad 6: Net-(Q3A-C) -> /amplifier_left/IPS_L
- Q6 pad 1: Net-(Q3A-C) -> /amplifier_left/IPS_L
- Q6 pad 2: Net-(Q6-E) -> /amplifier_left/VAS_DARL_L
- Q6 pad 3: GND -> /amplifier_left/V_{bias}-_L
- Q7 pad 3: /amplifier_left/CC_VAS -> /amplifier_left/CC_VAS_L
- Q8 pad 1: /amplifier_left/V_{bias}B -> /amplifier_left/V_{bias}B_L
- Q8 pad 2: /amplifier_left/V_{bias}- -> /amplifier_left/V_{bias}+_L
- Q8 pad 3: /amplifier_left/V_{bias}+ -> +25V
- Q9 pad 1: Net-(Q6-E) -> /amplifier_left/V_{bias}-_L
- Q9 pad 2: Net-(Q9-E) -> -25V
- Q9 pad 3: /amplifier_left/V_{bias}- -> -25V
- R1 pad 1: Net-(U1-POPGUARD/TSTO) -> VBUS
- R1 pad 2: VBUS -> /POPGUARD
- R10 pad 1: Net-(Q2B-E) -> unconnected-(R10-Pad1)
- R10 pad 2: unconnected-(R10-Pad2) -> Net-(Q2A-B)
- R11 pad 1: Net-(K1-Pad10) -> Net-(Q2A-B)
- R11 pad 2: GND -> Net-(Q1-C)
- R12 pad 1: Net-(K1-Pad3) -> Net-(Q2B-E)
- R12 pad 2: GND -> unconnected-(R12-Pad2)
- R13 pad 1: Net-(C16-Pad2) -> /DAC_L
- R13 pad 2: /OUT_L -> Net-(C16-Pad2)
- R14 pad 1: Net-(C17-Pad2) -> GND
- R14 pad 2: /OUT_R -> /amplifier_left/INPUT_L
- R15 pad 2: Net-(Q3A-B) -> Net-(Q4A-C)
- R16 pad 1: GND -> -20Vreg
- R16 pad 2: Net-(Q4A-C) -> Net-(Q5A-E)
- R17 pad 1: -20Vreg -> Net-(Q3A-E)
- R17 pad 2: Net-(Q5A-E) -> Net-(R17-Pad2)
- R18 pad 1: Net-(Q3A-E) -> Net-(R17-Pad2)
- R18 pad 2: Net-(R18-Pad2) -> /amplifier_left/CC_IPS_L
- R19 pad 1: Net-(R18-Pad2) -> Net-(Q4A-B)
- R19 pad 2: /amplifier_left/CC_IPS -> +20Vreg
- R2 pad 1: /OUT_L -> GND
- R2 pad 2: /DC_LP_L -> /AMP_L
- R20 pad 1: Net-(Q4A-B) -> Net-(R20-Pad1)
- R20 pad 2: +20Vreg -> /amplifier_left/CC_IPS_L
- R21 pad 1: Net-(R21-Pad1) -> Net-(R20-Pad1)
- R21 pad 2: /amplifier_left/CC_IPS -> Net-(Q3B-E)
- R22 pad 1: Net-(R21-Pad1) -> -20Vreg
- R22 pad 2: Net-(Q3B-E) -> Net-(Q5B-E)
- R23 pad 1: -20Vreg -> GND
- R23 pad 2: Net-(Q5B-E) -> /amplifier_left/FB_L
- R24 pad 1: GND -> /amplifier_left/FB_L
- R24 pad 2: /amplifier_left/FB -> /AMP_L
- R25 pad 1: /amplifier_left/FB -> -20Vreg
- R25 pad 2: /AMP_L -> /amplifier_left/VAS_DARL_L
- R26 pad 1: -20Vreg -> GND
- R26 pad 2: Net-(Q6-E) -> Net-(Q7A-C)
- R27 pad 1: GND -> /amplifier_left/V_{bias}B_L
- R27 pad 2: Net-(Q7A-C) -> /amplifier_left/CC_VAS_L
- R28 pad 1: /amplifier_left/V_{bias}B -> Net-(R28-Pad1)
- R28 pad 2: /amplifier_left/CC_VAS -> /amplifier_left/V_{bias}B_L
- R29 pad 1: Net-(R29-Pad1) -> Net-(Q7A-B)
- R29 pad 2: /amplifier_left/V_{bias}B -> +20Vreg
- R3 pad 1: /OUT_R -> GND
- R3 pad 2: /DC_LP_R -> /AMP_R
- R30 pad 1: Net-(Q7A-B) -> /amplifier_left/CC_VAS_L
- R30 pad 2: +20Vreg -> /amplifier_left/V_{bias}+_L
- R31 pad 1: /amplifier_left/CC_VAS -> -20Vreg
- R31 pad 2: /amplifier_left/V_{bias}+ -> Net-(Q6B-E)
- R32 pad 1: -20Vreg -> /AMP_L
- R32 pad 2: Net-(Q9-E) -> /amplifier_left/V_{OPS}+_L
- R33 pad 1: Net-(D9-C/A) -> /amplifier_left/V_{OPS}-_L
- R33 pad 2: /amplifier_left/V_{OPS}+ -> /AMP_L
- R34 pad 1: /amplifier_left/V_{OPS}- -> /amplifier_left/V_{q}+_L
- R34 pad 2: Net-(D9-C/A) -> /AMP_L
- R35 pad 1: /amplifier_left/V_{q}+ -> /AMP_L
- R35 pad 2: Net-(D9-C/A) -> /amplifier_left/V_{q}-_L
- R36 pad 1: Net-(D9-C/A) -> /amplifier_left/ZOBEL_L
- R36 pad 2: /amplifier_left/V_{q}- -> /AMP_L
- R38 pad 2: Net-(Q14A-B) -> /amplifier_right/INPUT_R
- R39 pad 2: Net-(Q15A-C) -> Net-(Q13A-C)
- R4 pad 1: Net-(C14-Pad2) -> /OUT_L
- R4 pad 2: /AMP_L -> /DC_LP_L
- R40 pad 2: Net-(Q16A-E) -> Net-(Q14A-E)
- R41 pad 1: Net-(Q14A-E) -> Net-(Q12A-E)
- R42 pad 2: /amplifier_right/CC_IPS -> /amplifier_right/CC_IPS_R
- R43 pad 1: Net-(Q15A-B) -> Net-(Q13A-B)
- R44 pad 2: /amplifier_right/CC_IPS -> /amplifier_right/CC_IPS_R
- R45 pad 2: Net-(Q14B-E) -> Net-(Q12B-E)
- R46 pad 2: Net-(Q16B-E) -> Net-(Q14B-E)
- R47 pad 2: /amplifier_right/FB -> /amplifier_right/FB_L
- R48 pad 1: /amplifier_right/FB -> /amplifier_right/FB_L
- R49 pad 2: Net-(Q17-E) -> /amplifier_right/VAS_DARL_R
- R5 pad 1: Net-(C15-Pad2) -> /OUT_R
- R5 pad 2: /AMP_R -> /DC_LP_R
- R50 pad 2: Net-(Q18A-C) -> Net-(Q16A-C)
- R51 pad 1: /amplifier_right/V_{bias}B -> /amplifier_right/V_{bias}B_R
- R51 pad 2: /amplifier_right/CC_VAS -> /amplifier_right/CC_VAS_R
- R52 pad 2: /amplifier_right/V_{bias}B -> /amplifier_right/V_{bias}B_R
- R53 pad 1: Net-(Q18A-B) -> Net-(Q16A-B)
- R54 pad 1: /amplifier_right/CC_VAS -> /amplifier_right/CC_VAS_R
- R54 pad 2: /amplifier_right/V_{bias}+ -> /amplifier_right/V_{bias}+_R
- R55 pad 2: Net-(Q20-E) -> Net-(Q15B-E)
- R56 pad 1: Net-(D10-C/A) -> /AMP_R
- R56 pad 2: /amplifier_right/V_{OPS}+ -> /amplifier_right/V_{OPS}+_R
- R57 pad 1: /amplifier_right/V_{OPS}- -> /amplifier_right/V_{OPS}-_R
- R57 pad 2: Net-(D10-C/A) -> /AMP_R
- R58 pad 1: /amplifier_right/V_{q}+ -> /amplifier_right/V_{q}+_R
- R58 pad 2: Net-(D10-C/A) -> /AMP_R
- R59 pad 1: Net-(D10-C/A) -> /AMP_R
- R59 pad 2: /amplifier_right/V_{q}- -> /amplifier_right/V_{q}-_R
- R6 pad 2: /AMP_L -> /RLY_NC_L
- R7 pad 2: /AMP_R -> /RLY_NC_R
- R8 pad 1: unconnected-(R8-Pad1) -> /PROT_ARC_L
- R8 pad 2: Net-(Q2A-B) -> /OUT_L
- R9 pad 1: Net-(Q2A-B) -> /PROT_ARC_R
- R9 pad 2: Net-(Q1-C) -> /OUT_R
- RV1 pad 1: /DAC_L -> Net-(C17-Pad2)
- RV1 pad 2: Net-(C18-Pad1) -> /amplifier_left/INPUT_L
- RV1 pad 4: /DAC_R -> Net-(C26-Pad2)
- RV1 pad 5: Net-(C23-Pad1) -> /amplifier_right/INPUT_R
- RV2 pad 1: Net-(R18-Pad2) -> Net-(R17-Pad2)
- RV2 pad 2: /amplifier_left/CC_IPS -> /amplifier_left/CC_IPS_L
- RV2 pad 3: Net-(R21-Pad1) -> Net-(R20-Pad1)
- RV3 pad 1: Net-(R29-Pad1) -> Net-(R28-Pad1)
- RV3 pad 2: /amplifier_left/V_{bias}- -> /amplifier_left/V_{bias}-_L
- RV3 pad 3: /amplifier_left/V_{bias}- -> /amplifier_left/V_{bias}-_L
- RV4 pad 2: /amplifier_right/CC_IPS -> /amplifier_right/CC_IPS_R
- RV5 pad 2: /amplifier_right/V_{bias}- -> /amplifier_right/V_{bias}-_R
- RV5 pad 3: /amplifier_right/V_{bias}- -> /amplifier_right/V_{bias}-_R
- U1 pad 20: Net-(U1-VQ) -> /VQ
- U1 pad 6: Net-(U1-VD_FILT) -> /VD_FILT
- U1 pad 8: Net-(U1-POPGUARD/TSTO) -> /POPGUARD
Other:
- board size 90 x 99 mm -> 88 x 99 mm
