File: kicad/front_plate/front_plate.kicad_pcb (KiCad board)
At the start: 2 copper layers, 103 x 53 mm, 11 parts, among them U2 TL431, U3 TL431

Commit message: commit
Parts:
- removed U3: TL431, Package_TO_SOT_SMD:SOT-23-3
- added D2: RED, library:LED_Harvatek_B2601, B.Cu at (102.5, 56.6)
- added D5: BLUE, library:LED_Harvatek_B2601, B.Cu at (114.5, 56.6)
- added G***: LOGO, library:USB-logo, F.Cu at (114.5, 52.0)
- added G***: LOGO, library:DC-logo, F.Cu at (102.5, 52.2)
- added R8: 1k5, Resistor_SMD:R_1206_3216Metric_Pad1.30x1.75mm_HandSolder, B.Cu at (114.1, 39.6)
- added R9: 1k5, Resistor_SMD:R_1206_3216Metric_Pad1.30x1.75mm_HandSolder, B.Cu at (117.3, 39.6)
- added SW1: SW_SPST, library:Switch_E-Switch_PB-1973_Cutout, F.Cu at (73.5, 56.5)
- added U1: TL431, Package_TO_SOT_SMD:SOT-23-3, B.Cu at (91.6, 45.1)
- C1, C2, R1, R2, R3, R4, R5, R6, R7, U2: moved to B.Cu
- moved R7 38.0 mm to (110.8, 39.6), turned to -90 degrees
- moved R6 33.4 mm to (107.5, 39.6), turned to -90 degrees
- moved R5 28.8 mm to (104.2, 39.6), turned to -90 degrees
- moved C2 25.7 mm to (110.3, 45.6), turned to -90 degrees
- moved R4 24.2 mm to (100.9, 39.6), turned to -90 degrees
- moved C1 21.4 mm to (107.0, 45.6), turned to -90 degrees
- moved R3 19.7 mm to (97.6, 39.6), turned to -90 degrees
- moved R2 15.3 mm to (94.3, 39.6), turned to -90 degrees
- moved R1 11.0 mm to (91.0, 39.6), turned to -90 degrees
- moved U2 10.2 mm to (96.1, 45.1), turned to -90 degrees
Connections:
- net GNDD renamed GND
- R5 pad 1: Net-(U3-K) -> Net-(U2-K)
- U2 pad 1: /V_{high} -> /V_{low}
- U2 pad 3: Net-(Q1-B) -> Net-(U2-K)
Routing:
- net (no net): vias 1 -> 0
Other:
- outline, holes or cut-outs redrawn

Commit message: commit
Parts:
- removed C1, C2: 10u, Capacitor_SMD:C_1206_3216Metric_Pad1.33x1.80mm_HandSolder
- removed D2: RED, library:LED_Harvatek_B2601
- removed D5: BLUE, library:LED_Harvatek_B2601
- removed the G*** at (102.5, 52.2)
- removed R7: 1k8, Resistor_SMD:R_1206_3216Metric_Pad1.30x1.75mm_HandSolder
- removed R8, R9: 1k5, Resistor_SMD:R_1206_3216Metric_Pad1.30x1.75mm_HandSolder
- removed SW1: SW_SPST, library:Switch_E-Switch_PB-1973_Cutout
- removed U1, U2: TL431, Package_TO_SOT_SMD:SOT-23-3
- added D3: AMBER, library:LED_Harvatek_B2601, B.Cu at (106.6, 49.0)
- added D7: AMBER, library:LED_Harvatek_B2601, B.Cu at (96.4, 49.0)
- added J1: Conn_01x04, Connector_PinSocket_2.54mm:PinSocket_1x04_P2.54mm_Vertical_SMD_Pin1Left, B.Cu at (82.8, 55.6)
- added Q1: BCM56DS, Package_SO:SC-74-6_1.5x2.9mm_P0.95mm, B.Cu at (108.1, 37.1)
- added Q2: BCM56DS, Package_SO:SC-74-6_1.5x2.9mm_P0.95mm, B.Cu at (108.1, 41.6)
- R1: value 10k -> 47k
- R2, R5: value 1k5 -> 2k2
- R3: value 100k -> 10k
- R4: value 1k8 -> 2k2
- R6: value 10k -> 4k3
- moved R1 23.4 mm to (114.2, 36.6), turned to 180 degrees
- moved R2 19.9 mm to (114.2, 39.9), turned to 180 degrees
- moved G*** 19.0 mm to (96.5, 45.7)
- moved R3 17.0 mm to (114.2, 43.1), turned to 180 degrees
- moved R6 15.0 mm to (114.2, 53.0), turned to 180 degrees
- moved R4 15.0 mm to (114.2, 46.4), turned to 180 degrees
- moved R5 14.3 mm to (114.2, 49.7), turned to 180 degrees
Connections:
- net /V_{high} renamed /ANALOG
- R1 pad 2: unconnected-(R1-Pad2) -> +24V
- R3 pad 2: unconnected-(R3-Pad2) -> +24V
- R4 pad 2: Net-(D1-RK) -> +24V
- R5 pad 2: Net-(D1-GK) -> +24V
- R6 pad 1: /V_{low} -> /USB
- R6 pad 2: unconnected-(R6-Pad2) -> Net-(Q2A-B1)
Other:
- board size 103 x 53 mm -> 103 x 30.5 mm
