File: kicad/front_plate/front_plate.kicad_sch (KiCad schematic)
At the start: 25 parts, among them J1 Conn_01x06_Pin, Q1 NPN, U1 BH1682FVC, U2 TL431, U3 TL431

Commit message: commit
Parts:
- added R17 (x2): 1k5, Resistor_SMD:R_1206_3216Metric_Pad1.30x1.75mm_HandSolder, symbol Device:R
- added SW1: SW_SPST, library:Switch_E-Switch_PB-1973_Cutout, symbol Switch:SW_SPST
- D11: footprint (none) -> library:LED_Harvatek_B2601
- D11: footprint (none) -> library:LED_Harvatek_B2601; Digikey 3147-B2601UY--20D000323U1930CT-ND -> (none)
- D11: footprint (none) -> library:LED_Harvatek_B2601; Digikey 3147-B2601NG--20C000923U1930CT-ND -> (none)
- U3: renamed from U1; now not fitted; now left out of the parts list
- renumbered D5 to D1, U2 to U1, U3 to U2
Connections:
- net GNDD is gone; now on net GND: C6.2, C6.2, Q1.3 (E), R16.1, R16.1, U1.2 (A), U2.2 (A)
- net GND: now also J1.3 (Pin_3), R17.1, R17.1
- net +25V: now reaches J1.1 (Pin_1)
- net +25V: now also D1.2 (A), D11.2 (A), D11.2 (A), R17.2, R17.2, R17.2
- net -25V: now reaches J1.2 (Pin_2)
- net DC: now reaches J1.4 (Pin_4)
- net USB: now reaches J1.5 (Pin_5)
- net at D11.1 (K): now also R17.2 (x2)
- no-connect marks 1 -> 4
Other:
- note added: "100k should be smaller"
- note added: "From DAC Board"
- note added: "Power Switch"
- company: Jona Heinke -> Author: Jona Heinke
- moved on the sheet: C6, D1, D11, Q1, R16, R17, R21, R22, U1, U2

Commit message: commit
Parts:
- removed C6 (x2): 10u, Capacitor_SMD:C_1206_3216Metric_Pad1.33x1.80mm_HandSolder, symbol Device:C
- removed D11: BLUE, library:LED_Harvatek_B2601, symbol Device:LED
- removed D11: RED, library:LED_Harvatek_B2601, symbol Device:LED
- removed J1: Conn_01x06_Pin, symbol Connector:Conn_01x06_Pin
- removed Q1: NPN, symbol Simulation_SPICE:NPN
- removed R16, R17, R22: 1k5, Resistor_SMD:R_1206_3216Metric_Pad1.30x1.75mm_HandSolder, symbol Device:R
- removed R16, R21: 1k8, Resistor_SMD:R_1206_3216Metric_Pad1.30x1.75mm_HandSolder, symbol Device:R
- removed R17 (x2): 10k, Resistor_SMD:R_1206_3216Metric_Pad1.30x1.75mm_HandSolder, symbol Device:R
- removed R17: 100k, Resistor_SMD:R_1206_3216Metric_Pad1.30x1.75mm_HandSolder, symbol Device:R
- removed U2: TL431, Package_TO_SOT_SMD:SOT-23-3, symbol Reference_Voltage:TL431PK
- added D11 (x2): AMBER, library:LED_Harvatek_B2601, symbol Device:LED
- added J1: Conn_01x04, Connector_PinSocket_2.54mm:PinSocket_1x04_P2.54mm_Vertical_SMD_Pin1Left, symbol Connector_Generic:Conn_01x04
- added Q3 (x2): BCM56DS, Package_SO:SC-74-6_1.5x2.9mm_P0.95mm, symbol library:Dual-NPN
- added R17 (x2): 2k2, Resistor_SMD:R_1206_3216Metric_Pad1.30x1.75mm_HandSolder, symbol Device:R
- added R17: 10k, Resistor_SMD:R_1206_3216Metric_Pad1.30x1.75mm_HandSolder, symbol Device:R
- added R17: 47k, Resistor_SMD:R_1206_3216Metric_Pad1.30x1.75mm_HandSolder, symbol Device:R
- added R20: 4k3, Resistor_SMD:R_1206_3216Metric_Pad1.30x1.75mm_HandSolder, symbol Device:R
- D11: renamed from D1; now not fitted; now left out of the parts list
- R17: value 1k5 -> 2k2
- SW1: footprint library:Switch_E-Switch_PB-1973_Cutout -> (none)
- U2: renamed from U1; now not fitted; now left out of the parts list
- renumbered U3 to U1
Connections:
- net GND: now also J1.4 (Pin_4), Q3.4 (E2), Q3.4 (E2), Q3.5 (E1), R17.1; no longer R17.1, U2.2 (A)
- net USB: now also J1.2 (Pin_2), R20.1
- net +24V: now reaches R17.2
- net +24V: now also J1.1 (Pin_1), R17.2, R17.2, R17.2
- net +25V: no longer names the net of D11.2 (A)
- net V_{high}: no longer names the net of U2.1 (REF)
- new net: Q3.1 (B1), R20.2
- new net: Q3.3 (C2), Q3.5 (E1)
- new net: D11.1 (K), Q3.6 (C1)
- new net: Q3.2 (B2), Q3.2 (B2), Q3.6 (C1), R17.1
- new net: D11.2 (A), R17.1 (x2)
- new net: D11.1 (K), Q3.3 (C2)
- new net ANALOG: J1.3 (Pin_3), Q3.1 (B1), R17.1, R17.2
- no-connect marks 4 -> 2
Other:
- note added: "USB is 0-3.3V ANALOG is shorted to ground when plug is detected otherwise floating"
- note added: "missing cutout"
- note removed: "100k should be smaller"
- note removed: "DC detection"
- note removed: "LED Indicator"
- note removed: "TH=16.39V"
- note removed: "TH=19.17V"
- note removed: "USB detection"
- moved on the sheet: R17, SW1
